File: crocus.kicad_pcb (KiCad board)
At the start: 4 copper layers, 70.7 x 53.3 mm, 49 parts, among them J1 NEIGHBOR1, J2 NEIGHBOR2, J7 BONUS_ROW, P1 RP-SMA, P2 EXPANSION, T1 BALUN, U1 nRF24L01+, U2 PCA9674, Y1 XTAL

Commit message: adopt OSHWA convention for SPI signal names https://www.oshwa.org/a-resolution-to-redefine-spi-signal-names
Connections:
- net /MISO renamed /CIPO
- net /MISO_ALT1 renamed /CIPO_ALT1
- net /MOSI renamed /COPI
- net /MOSI_ALT1 renamed /COPI_ALT1
Other:
- board text added: "CIPO"
- board text added: "COPI"
- board text removed: "MISO"
- board text removed: "MOSI"
Changed lines of the file:
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@@
   (net 41 /CSN_ALT1)
   (net 42 /SCK)
-  (net 43 /MOSI)
-  (net 44 /MISO)
+  (net 43 /COPI)
+  (net 44 /CIPO)
   (net 45 "Net-(J2-Pad3)")
   (net 46 /INT)
@@
   (net 70 "Net-(J2-Pad28)")
   (net 71 "Net-(J2-Pad29)")
-  (net 72 /MOSI_ALT1)
+  (net 72 /COPI_ALT1)
   (net 73 "Net-(J2-Pad31)")
   (net 74 /SCK_ALT1)
@@
   (net 78 "Net-(J2-Pad36)")
   (net 79 "Net-(J2-Pad37)")
-  (net 80 /MISO_ALT1)
+  (net 80 /CIPO_ALT1)
   (net 81 /I2C0_SDA)
   (net 82 /I2C0_SCL)
@@
     (add_net /IREF)
     (add_net /IRQ)
-    (add_net /MISO)
-    (add_net /MISO_ALT1)
-    (add_net /MOSI)
-    (add_net /MOSI_ALT1)
+    (add_net /CIPO)
+    (add_net /CIPO_ALT1)
+    (add_net /COPI)
+    (add_net /COPI_ALT1)
     (add_net /P0)
     (add_net /P1)
@@
       (net 42 /SCK) (die_length -2147.483648))
     (pad 39 thru_hole circle (at 24.13 1.27) (size 1.524 1.524) (drill 1.016) (layers *.Cu *.Mask F.SilkS)
-      (net 43 /MOSI) (die_length 0.08382))
+      (net 43 /COPI) (die_length 0.08382))
     (pad 40 thru_hole circle (at 24.13 -1.27) (size 1.524 1.524) (drill 1.016) (layers *.Cu *.Mask F.SilkS)
-      (net 44 /MISO) (die_length 0.08382))
+      (net 44 /CIPO) (die_length 0.08382))
   )
   (module gsg-modules:HEADER-2x20 (layer C1F.Cu)
@@
       (net 71 "Net-(J2-Pad29)") (die_length 0.08382))
     (pad 30 thru_hole circle (at 11.43 -1.27) (size 1.524 1.524) (drill 1.016) (layers *.Cu *.Mask F.SilkS)
-      (net 72 /MOSI_ALT1) (die_length -2147.483648))
+      (net 72 /COPI_ALT1) (die_length -2147.483648))
     (pad 31 thru_hole circle (at 13.97 1.27) (size 1.524 1.524) (drill 1.016) (layers *.Cu *.Mask F.SilkS)
       (net 73 "Net-(J2-Pad31)") (die_length 0.08382))
@@
       (net 79 "Net-(J2-Pad37)") (die_length 0.08382))
     (pad 38 thru_hole circle (at 21.59 -1.27) (size 1.524 1.524) (drill 1.016) (layers *.Cu *.Mask F.SilkS)
-      (net 80 /MISO_ALT1) (die_length -2147.483648))
+      (net 80 /CIPO_ALT1) (die_length -2147.483648))
     (pad 39 thru_hole circle (at 24.13 1.27) (size 1.524 1.524) (drill 1.016) (layers *.Cu *.Mask F.SilkS)
       (net 81 /I2C0_SDA) (die_length 0.08382))
@@
       (net 42 /SCK) (die_length 0.08382))
     (pad 4 smd oval (at -2.2 0.5) (size 1.2 0.32) (layers C1F.Cu F.Paste F.Mask)
-      (net 43 /MOSI) (die_length -0.00254))
+      (net 43 /COPI) (die_length -0.00254))
     (pad 5 smd oval (at -2.2 1) (size 1.2 0.32) (layers C1F.Cu F.Paste F.Mask)
-      (net 44 /MISO) (die_length 0.08382))
+      (net 44 /CIPO) (die_length 0.08382))
     (pad 6 smd oval (at -1 2.2 90) (size 1.2 0.32) (layers C1F.Cu F.Paste F.Mask)
       (net 110 /IRQ) (die_length 0.08382))
@@
     (fp_arc (start -0.762 0) (end -0.762 0.6096) (angle 180) (layer F.SilkS) (width 0.15))
     (pad 1 smd oval (at -0.6477 0) (size 1.0922 0.8636) (layers C1F.Cu F.Mask)
-      (net 80 /MISO_ALT1) (solder_mask_margin 0.1016) (clearance 0.1778))
-    (pad 2 smd rect (at 0.3556 0) (size 0.508 0.8636) (layers C1F.Cu F.Mask)
-      (net 44 /MISO) (solder_mask_margin 0.1016) (clearance 0.1778))
-    (pad 1 smd rect (at -0.3556 0) (size 0.508 0.8636) (layers C1F.Cu F.Mask)
-      (net 80 /MISO_ALT1) (solder_mask_margin 0.1016) (clearance 0.1778))
-    (pad 2 smd oval (at 0.6477 0) (size 1.0922 0.8636) (layers C1F.Cu F.Mask)
-      (net 44 /MISO))
+      (net 80 /CIPO_ALT1) (solder_mask_margin 0.1016) (clearance 0.1778))
+    (pad 2 smd rect (at 0.3556 0) (size 0.508 0.8636) (layers C1F.Cu F.Mask)
+      (net 44 /CIPO) (solder_mask_margin 0.1016) (clearance 0.1778))
+    (pad 1 smd rect (at -0.3556 0) (size 0.508 0.8636) (layers C1F.Cu F.Mask)
+      (net 80 /CIPO_ALT1) (solder_mask_margin 0.1016) (clearance 0.1778))
+    (pad 2 smd oval (at 0.6477 0) (size 1.0922 0.8636) (layers C1F.Cu F.Mask)
+      (net 44 /CIPO))
   )
   (module gsg-modules:0603-JUMPER (layer C1F.Cu)
@@
     (fp_arc (start -0.762 0) (end -0.762 0.6096) (angle 180) (layer F.SilkS) (width 0.15))
     (pad 1 smd oval (at -0.6477 0) (size 1.0922 0.8636) (layers C1F.Cu F.Mask)
-      (net 72 /MOSI_ALT1) (solder_mask_margin 0.1016) (clearance 0.1778))
-    (pad 2 smd rect (at 0.3556 0) (size 0.508 0.8636) (layers C1F.Cu F.Mask)
-      (net 43 /MOSI) (solder_mask_margin 0.1016) (clearance 0.1778))
-    (pad 1 smd rect (at -0.3556 0) (size 0.508 0.8636) (layers C1F.Cu F.Mask)
-      (net 72 /MOSI_ALT1) (solder_mask_margin 0.1016) (clearance 0.1778))
-    (pad 2 smd oval (at 0.6477 0) (size 1.0922 0.8636) (layers C1F.Cu F.Mask)
-      (net 43 /MOSI))
+      (net 72 /COPI_ALT1) (solder_mask_margin 0.1016) (clearance 0.1778))
+    (pad 2 smd rect (at 0.3556 0) (size 0.508 0.8636) (layers C1F.Cu F.Mask)
+      (net 43 /COPI) (solder_mask_margin 0.1016) (clearance 0.1778))
+    (pad 1 smd rect (at -0.3556 0) (size 0.508 0.8636) (layers C1F.Cu F.Mask)
+      (net 72 /COPI_ALT1) (solder_mask_margin 0.1016) (clearance 0.1778))
+    (pad 2 smd oval (at 0.6477 0) (size 1.0922 0.8636) (layers C1F.Cu F.Mask)
+      (net 43 /COPI))
   )
   (module gsg-modules:0603-JUMPER (layer C1F.Cu)
@@
       (net 1 GND))
   )
-  (gr_text MOSI (at 145.796 101.6) (layer F.SilkS)
+  (gr_text COPI (at 145.796 101.6) (layer F.SilkS)
     (effects (font (size 0.635 0.508) (thickness 0.1016)))
   )
@@
     (effects (font (size 0.635 0.508) (thickness 0.1016)))
   )
-  (gr_text MISO (at 145.796 103.632) (layer F.SilkS)
+  (gr_text CIPO (at 145.796 103.632) (layer F.SilkS)
     (effects (font (size 0.635 0.508) (thickness 0.1016)))
   )
@@
     (effects (font (size 0.635 0.508) (thickness 0.1016)))
   )
-  (gr_text MISO (at 172.72 116.84) (layer F.SilkS)
-    (effects (font (size 0.635 0.508) (thickness 0.1016)))
-  )
-  (gr_text MOSI (at 172.72 119.38) (layer F.SilkS)
-    (effects (font (size 0.635 0.508) (thickness 0.1016)))
-  )
+  (gr_text CIPO (at 172.72 116.84) (layer F.SilkS)
+    (effects (font (size 0.635 0.508) (thickness 0.1016)))
+  )
+  (gr_text COPI (at 172.72 119.38) (layer F.SilkS)
+    (effects (font (size 0.635 0.508) (thickness 0.1016)))
+  )
