File: crocus.sch (KiCad schematic (older format))
At the start: 49 parts, among them J1 NEIGHBOR1, J2 NEIGHBOR2, J7 BONUS_ROW, P1 RP-SMA, P2 EXPANSION, T1 BALUN, U1 nRF24L01+, U2 PCA9674, Y1 XTAL

Commit message: adopt OSHWA convention for SPI signal names https://www.oshwa.org/a-resolution-to-redefine-spi-signal-names
Connections:
- net MISO renamed CIPO
- net MISO_ALT1 renamed CIPO_ALT1
- net MOSI renamed COPI
- net MOSI_ALT1 renamed COPI_ALT1
Other:
- note added: "CS/P1_20"
- note removed: "SSEL/P1_20"
Changed lines of the file:
@@
 $EndComp
 Text Label 9850 6600 2    40   ~ 0
-MISO
+CIPO
 Text Label 8950 6600 0    40   ~ 0
-MOSI
+COPI
 Text Label 9850 6500 2    40   ~ 0
 SCK
@@
 P1_19
 Text Notes 8800 6500 2    40   ~ 0
-SSEL/P1_20
+CS/P1_20
 Text Label 9950 4000 2    40   ~ 0
 I2C0_SCL
@@
 SCK
 Text Label 5000 3750 0    40   ~ 0
-MOSI
+COPI
 Text Label 5000 3850 0    40   ~ 0
-MISO
+CIPO
 $Comp
 L Crystal Y1
@@
 P3_3
 Text Label 10000 3900 2    40   ~ 0
-MISO_ALT1
+CIPO_ALT1
 Text Label 10000 3500 2    40   ~ 0
-MOSI_ALT1
+COPI_ALT1
 Text Notes 10050 3500 0    40   ~ 0
 P3_7
@@
 	4500 5250 4150 5250
 Text Label 4500 5600 2    40   ~ 0
-MOSI_ALT1
+COPI_ALT1
 Text Label 3550 5600 0    40   ~ 0
-MOSI
+COPI
 Wire Wire Line
 	3550 5600 3750 5600
@@
 	4500 5600 4150 5600
 Text Label 4500 5900 2    40   ~ 0
-MISO_ALT1
+CIPO_ALT1
 Text Label 3550 5900 0    40   ~ 0
-MISO
+CIPO
 Wire Wire Line
 	3550 5900 3750 5900
